Commit message: study: controller 설정 추가

File: bumperbot_ws/src/bumperbot_description/urdf/bumperbot_gazebo.xacro (robot description, xacro)
@@ -1,5 +1,5 @@
 <?xml version="1.0"?>
-<robot name="bumperbot" xmlns:xacro="http://www.ros.org/wiki/xacro">
-  <gazebo reference="whell_right_link">
+<robot xmlns:xacro="http://www.ros.org/wiki/xacro" name="bumperbot">
+  <gazebo reference="wheel_right_link">
     <!-- 마찰력 -->
     <mu1>100000000000000.0</mu1>
@@ -13,5 +13,5 @@
     <fdirl>1 0 0</fdirl>
   </gazebo>
-  <gazebo reference="whell_left_link">
+  <gazebo reference="wheel_left_link">
     <mu1>100000000000000.0</mu1>
     <mu2>100000000000000.0</mu2>
@@ -49,10 +49,10 @@
     <xacro:if value="$(arg is_ignition)">
       <plugin filename="ign_ros2_control-system" name="ign_ros2_control::IgnitionROS2ControlPlugin">
-        <parmeters></parmeters>
+        <parmeters>$(find bumperbot_controller)/config/bumperbot_controllers.yaml</parmeters>
       </plugin>
     </xacro:if>
     <xacro:unless value="$(arg is_ignition)">
       <plugin filename="gz_ros2_control-system" name="gz_ros2_control::GazeboSimROS2ControlPlugin">
-        <parameters></parameters>
+        <parameters>$(find bumperbot_controller)/config/bumperbot_controllers.yaml</parameters>
       </plugin>
     </xacro:unless>

File: bumperbot_ws/src/bumperbot_description/urdf/bumperbot_ros2_control.xacro (robot description, xacro)
@@ -1,37 +1,35 @@
 <?xml version="1.0"?>
-<robot name="bumperbot" xmlns:xacro="http://www.ros.org/wiki/xacro">
-  <ros2_control name="RobotSystem" type="system">
-    <xacro:if value="$(arg is_ignition)">
-      <hardware>
-        <plugin>ign_ros2_control/IgnitionSystem</plugin>
-      </hardware>
-    </xacro:if>
-    <xacro:unless value="$(arg is_ignition)">
-      <hardware>
-        <plugin>gz_ros2_control/GaziboSimSystem</plugin>
-      </hardware>
-    </xacro:unless>
-    <!-- define interface joint of robot -->
-    <joint name="wheel_right_joint">
-      <!-- how to write hardware -->
-      <command_interface name="velocity">
-        <param name="min">-1</param>
-        <param name="max">1</param>
-      </command_interface>
-      <!-- how to read hardware -->
-      <state_interface name="position"/>
-      <state_interface name="velocity"/>
-    </joint>
-        <!-- define interface joint of robot -->
+<robot xmlns:xacro="http://www.ros.org/wiki/xacro" name="bumperbot">
+    <ros2_control name="RobotSystem" type="system">
+        <!-- ros2_control Gazebo -->
+        <!-- ROS 2 Humble -->
+        <xacro:if value="$(arg is_ignition)">
+            <hardware>
+                <plugin>ign_ros2_control/IgnitionSystem</plugin>
+            </hardware>
+        </xacro:if>
+        <!-- ROS 2 Iron or above -->
+        <xacro:unless value="$(arg is_ignition)">
+            <hardware>
+                <plugin>gz_ros2_control/GazeboSimSystem</plugin>
+            </hardware>
+        </xacro:unless>
+        <!-- ros2_control Common Interfaces -->
+        <joint name="wheel_right_joint">
+            <command_interface name="velocity">
+              <param name="min">-1</param>
+              <param name="max">1</param>
+            </command_interface>
+            <state_interface name="position" />
+            <state_interface name="velocity" />
+        </joint>
         <joint name="wheel_left_joint">
-          <!-- how to write hardware -->
-          <command_interface name="velocity">
-            <param name="min">-1</param>
-            <param name="max">1</param>
-          </command_interface>
-          <!-- how to read hardware -->
-          <state_interface name="position"/>
-          <state_interface name="velocity"/>
+            <command_interface name="velocity">
+              <param name="min">-1</param>
+              <param name="max">1</param>
+            </command_interface>
+            <state_interface name="position" />
+            <state_interface name="velocity" />
         </joint>
-  </ros2_control>
+    </ros2_control>
 </robot>
