Commit message: study: parameter / launch 실습

File: bumperbot_ws/src/bumperbot_description/urdf/bumperbot.urdf.xacro (robot description, xacro)
@@ -54,6 +54,6 @@
   <link name="caster_front_link">
     <visual>
+      <origin rpy="0.0 0.0 0.0" xyz="0 0 0" />
       <geometry>
-        <origin rpy="0.0 0.0 0.0" xyz="0 0 0" />
         <mesh filename="package://bumperbot_description/meshes/caster_front_link.STL"/>
       </geometry>
@@ -65,15 +65,15 @@
     <origin rpy="0.0 0.0 0.0" xyz="0.04755 0.0 -0.0275"/>
   </joint>
-  <link name="caster_lear_link">
+  <link name="caster_rear_link">
     <visual>
+      <origin rpy="0.0 0.0 0.0" xyz="0 0 0" />
       <geometry>
-        <origin rpy="0.0 0.0 0.0" xyz="0 0 0" />
-        <mesh filename="package://bumperbot_description/meshes/caster_lear_link.STL"/>
+        <mesh filename="package://bumperbot_description/meshes/caster_rear_link.STL"/>
       </geometry>
     </visual>
   </link>
-  <joint name="caster_lear_joint" type="fixed">
+  <joint name="caster_rear_joint" type="fixed">
     <parent link="base_link"/>
-    <child link="caster_lear_link"/>
+    <child link="caster_rear_link"/>
     <origin rpy="0.0 0.0 0.0" xyz="-0.04755 0.0 -0.0275"/>
   </joint>

Commit message: study: can.STL을 bumperbot 위에 올리기 실습

File: bumperbot_ws/src/bumperbot_description/urdf/bumperbot.urdf.xacro (robot description, xacro)
@@ -7,22 +7,22 @@
     <visual>
       <!-- 시각 측면에서 메시의 각도 및 좌표. rpy = 각도, xyz = 좌표 -->
-      <origin rpy="0.0 0.0 0.0" xyz="0.0 0.0 0.0"/>
+      <origin rpy="0.0 0.0 0.0" xyz="0.0 0.0 0.0" />
       <geometry>
         <!-- 메시 파일 위치 -->
-        <mesh filename="package://bumperbot_description/meshes/base_link.STL"/>
+        <mesh filename="package://bumperbot_description/meshes/base_link.STL" />
       </geometry>
     </visual>
   </link>
   <joint name="base_joint" type="fixed">
-    <parent link="base_footprint"/>
-    <child link="base_link"/>
+    <parent link="base_footprint" />
+    <child link="base_link" />
     <!-- parent에 대한 child의 상대 각도 / 위치 -->
-    <origin rpy="0.0 0.0 0.0" xyz="0.0 0.0 0.033"/>
+    <origin rpy="0.0 0.0 0.0" xyz="0.0 0.0 0.033" />
   </joint>
   <link name="wheel_right_link">
     <visual>
-      <origin rpy="1.57 0 0" xyz="0 0 0"/>
+      <origin rpy="1.57 0 0" xyz="0 0 0" />
       <geometry>
-        <mesh filename="package://bumperbot_description/meshes/wheel_right_link.STL"/>
+        <mesh filename="package://bumperbot_description/meshes/wheel_right_link.STL" />
       </geometry>
     </visual>
@@ -31,14 +31,14 @@
   <joint name="wheel_right_joint" type="continuous">
     <parent link="base_link" />
-    <child link="wheel_right_link"/>
+    <child link="wheel_right_link" />
     <!-- y축 -->
-    <axis xyz="0 1 0"/>
-    <origin rpy="0.0 0.0 0.0" xyz="0.0 -0.07 0.0"/>
+    <axis xyz="0 1 0" />
+    <origin rpy="0.0 0.0 0.0" xyz="0.0 -0.07 0.0" />
   </joint>
   <link name="wheel_left_link">
     <visual>
-      <origin rpy="-1.57 0 0" xyz="0 0 0"/>
+      <origin rpy="-1.57 0 0" xyz="0 0 0" />
       <geometry>
-        <mesh filename="package://bumperbot_description/meshes/wheel_left_link.STL"/>
+        <mesh filename="package://bumperbot_description/meshes/wheel_left_link.STL" />
       </geometry>
     </visual>
@@ -47,8 +47,8 @@
   <joint name="wheel_left_joint" type="continuous">
     <parent link="base_link" />
-    <child link="wheel_left_link"/>
+    <child link="wheel_left_link" />
     <!-- y축 -->
-    <axis xyz="0 1 0"/>
-    <origin rpy="0.0 0.0 0.0" xyz="0.0 0.07 0.0"/>
+    <axis xyz="0 1 0" />
+    <origin rpy="0.0 0.0 0.0" xyz="0.0 0.07 0.0" />
   </joint>
   <link name="caster_front_link">
@@ -56,12 +56,12 @@
       <origin rpy="0.0 0.0 0.0" xyz="0 0 0" />
       <geometry>
-        <mesh filename="package://bumperbot_description/meshes/caster_front_link.STL"/>
+        <mesh filename="package://bumperbot_description/meshes/caster_front_link.STL" />
       </geometry>
     </visual>
   </link>
   <joint name="caster_front_joint" type="fixed">
-    <parent link="base_link"/>
-    <child link="caster_front_link"/>
-    <origin rpy="0.0 0.0 0.0" xyz="0.04755 0.0 -0.0275"/>
+    <parent link="base_link" />
+    <child link="caster_front_link" />
+    <origin rpy="0.0 0.0 0.0" xyz="0.04755 0.0 -0.0275" />
   </joint>
   <link name="caster_rear_link">
@@ -69,12 +69,26 @@
       <origin rpy="0.0 0.0 0.0" xyz="0 0 0" />
       <geometry>
-        <mesh filename="package://bumperbot_description/meshes/caster_rear_link.STL"/>
+        <mesh filename="package://bumperbot_description/meshes/caster_rear_link.STL" />
       </geometry>
     </visual>
   </link>
   <joint name="caster_rear_joint" type="fixed">
+    <parent link="base_link" />
+    <child link="caster_rear_link" />
+    <origin rpy="0.0 0.0 0.0" xyz="-0.04755 0.0 -0.0275" />
+  </joint>
+  <link name="can_link">
+    <visual>
+      <origin rpy="1.57 0.0 0.0" xyz="-0.0321 0.0321 0.0" />
+      <geometry>
+        <mesh filename="package://bumperbot_description/meshes/can.STL"/>
+      </geometry>
+    </visual>
+  </link>
+  <joint name="can_joint" type="fixed">
     <parent link="base_link"/>
-    <child link="caster_rear_link"/>
-    <origin rpy="0.0 0.0 0.0" xyz="-0.04755 0.0 -0.0275"/>
+    <child link="can_link"/>
+    <!-- checked by blender -->
+    <origin rpy="0.0 0.0 0.0" xyz="0 0 0.08"/>
   </joint>
 </robot>

Commit message: study: urdf 모델에 물리 요소 추가, gazebo 연동

File: bumperbot_ws/src/bumperbot_description/urdf/bumperbot.urdf.xacro (robot description, xacro)
@@ -1,8 +1,16 @@
 <?xml version="1.0"?>
 <robot xmlns:xacro="http://www.ros.org/wiki/xacro" name="bumperbot">
+  <xacro:include filename="$(find bumperbot_description)/urdf/bumperbot_gazebo.xacro"/>
   <!-- 외부 - 로봇 사이를 연결하는 일종의 인터페이스 역할 -->
   <link name="base_footprint" />
   <!-- 실제 로봇 역할 -->
   <link name="base_link">
+    <inertial>
+      <origin xyz="0 0 0.04" rpy="0.0 0.25 0.3" />
+      <mass value="8.2573504e-01" />
+      <inertia ixx="2.2124416e-02" ixy="-1.2294101e-04" ixz="3.4938785e-04"
+        iyy="2.1193702e-02" iyz="-5.0120904e-05" izz="2.0064271e-02"
+      />
+    </inertial>
     <visual>
       <!-- 시각 측면에서 메시의 각도 및 좌표. rpy = 각도, xyz = 좌표 -->
@@ -13,4 +21,11 @@
       </geometry>
     </visual>
+    <collision>
+      <origin rpy="0.0 0.0 0.0" xyz="0.0 0.0 0.0" />
+      <geometry>
+        <!-- 메시 파일 위치 -->
+        <mesh filename="package://bumperbot_description/meshes/base_link.STL" />
+      </geometry>
+    </collision>
   </link>
   <joint name="base_joint" type="fixed">
@@ -21,4 +36,11 @@
   </joint>
   <link name="wheel_right_link">
+    <inertial>
+      <origin xyz="0 -0.014 0" rpy="0 0 0" />
+      <mass value="0.0530086090966721" />
+      <inertia ixx="1.88176298336665E-05" ixy="-4.8444933029987E-10" ixz="1.88163708851143E-08"
+        iyy="3.11510738647764E-05" iyz="-6.93560663069607E-11" izz="1.8801969558182E-05"
+      />
+    </inertial>
     <visual>
       <origin rpy="1.57 0 0" xyz="0 0 0" />
@@ -27,4 +49,11 @@
       </geometry>
     </visual>
+    <!-- collider != mesh -->
+    <collision>
+      <origin rpy="1.57 0 0" xyz="0 -0.015 0" />
+      <geometry>
+        <sphere radius="0.033" />
+      </geometry>
+    </collision>
   </link>
   <!-- continous => rollable -->
@@ -37,4 +66,11 @@
   </joint>
   <link name="wheel_left_link">
+    <inertial>
+      <origin xyz="0 0.014 0" rpy="0 0 0" />
+      <mass value="0.0530086043217644" />
+      <inertia ixx="1.8792911368909E-05"  ixy="3.31256392204584E-10" ixz="-1.14082001662767E-08"
+               iyy="3.11510738759073E-05" iyz="-3.60499245082192E-10"
+               izz="1.88266886146847E-05" />
+    </inertial>
     <visual>
       <origin rpy="-1.57 0 0" xyz="0 0 0" />
@@ -43,4 +79,10 @@
       </geometry>
     </visual>
+    <collision>
+      <origin rpy="1.57 0 0" xyz="0 0.015 0" />
+      <geometry>
+        <sphere radius="0.033" />
+      </geometry>
+    </collision>
   </link>
   <!-- continous => rollable -->
@@ -53,4 +95,7 @@
   </joint>
   <link name="caster_front_link">
+    <inertia ixx="7.23075276010246E-11" ixy="-6.10956883467859E-16" ixz="2.22849693525031E-15"
+               iyy="3.8713793085917E-11"  iyz="2.93909858781952E-15"
+               izz="1.00967486676306E-10" />
     <visual>
       <origin rpy="0.0 0.0 0.0" xyz="0 0 0" />
@@ -59,4 +104,10 @@
       </geometry>
     </visual>
+    <collision>
+      <origin rpy="0 0 0" xyz="0 0 0" />
+      <geometry>
+        <sphere radius="0.005" />
+      </geometry>
+    </collision>
   </link>
   <joint name="caster_front_joint" type="fixed">
@@ -66,4 +117,7 @@
   </joint>
   <link name="caster_rear_link">
+    <inertia ixx="7.23075276010246E-11" ixy="-6.10956872363424E-16" ixz="2.22849693527207E-15"
+    iyy="3.87137930859167E-11" iyz="2.939098587861E-15"
+    izz="1.00967486676306E-10" />
     <visual>
       <origin rpy="0.0 0.0 0.0" xyz="0 0 0" />
@@ -72,4 +126,11 @@
       </geometry>
     </visual>
+    <!-- visual == volume. not all case. -->
+    <collision>
+      <origin rpy="0 0 0" xyz="0 0 0" />
+      <geometry>
+        <sphere radius="0.005" />
+      </geometry>
+    </collision>
   </link>
   <joint name="caster_rear_joint" type="fixed">
@@ -82,13 +143,13 @@
       <origin rpy="1.57 0.0 0.0" xyz="-0.0321 0.0321 0.0" />
       <geometry>
-        <mesh filename="package://bumperbot_description/meshes/can.STL"/>
+        <mesh filename="package://bumperbot_description/meshes/can.STL" />
       </geometry>
     </visual>
   </link>
   <joint name="can_joint" type="fixed">
-    <parent link="base_link"/>
-    <child link="can_link"/>
+    <parent link="base_link" />
+    <child link="can_link" />
     <!-- checked by blender -->
-    <origin rpy="0.0 0.0 0.0" xyz="0 0 0.08"/>
+    <origin rpy="0.0 0.0 0.0" xyz="0 0 0.08" />
   </joint>
 </robot>

Commit message: study: c++ controller 작성

File: bumperbot_ws/src/bumperbot_description/urdf/bumperbot.urdf.xacro (robot description, xacro)
@@ -1,33 +1,28 @@
 <?xml version="1.0"?>
-<robot xmlns:xacro="http://www.ros.org/wiki/xacro" name="bumperbot">
-  <!-- 적절한 ros2 control library를 가져오기 위한 변수. ros2 버전에 따라 다른 플러그인을 사용. -->
-  <xacro:arg name ="is_ignition" default="false"/>
-  <!-- gazebo params -->
-  <xacro:include filename="$(find bumperbot_description)/urdf/bumperbot_gazebo.xacro"/>
-  <!-- ros2 control lib -->
-  <xacro:include filename="$(find bumperbot_description)/urdf/bumperbot_ros2_control.xacro"/>
-  <!-- 외부 - 로봇 사이를 연결하는 일종의 인터페이스 역할 -->
-  <link name="base_footprint" />
-  <!-- 실제 로봇 역할 -->
+<robot name="bumperbot" xmlns:xacro="http://ros.org/wiki/xacro">
+  <!-- Start GZ or Ignition depending on ROS 2 Version -->
+  <xacro:arg name="is_ignition" default="true"/>
+  <!-- Include Gazebo Parameters -->
+  <xacro:include filename="$(find bumperbot_description)/urdf/bumperbot_gazebo.xacro" />
+  <!-- Include ros2_control Plugins -->
+  <xacro:include filename="$(find bumperbot_description)/urdf/bumperbot_ros2_control.xacro" />
+  <link name="base_footprint"/>
   <link name="base_link">
     <inertial>
       <origin xyz="0 0 0.04" rpy="0.0 0.25 0.3" />
-      <mass value="8.2573504e-01" />
+      <mass value="8.2573504e-01"/>
       <inertia ixx="2.2124416e-02" ixy="-1.2294101e-04" ixz="3.4938785e-04"
-        iyy="2.1193702e-02" iyz="-5.0120904e-05" izz="2.0064271e-02"
-      />
+               iyy="2.1193702e-02" iyz="-5.0120904e-05"
+               izz="2.0064271e-02" />
     </inertial>
     <visual>
-      <!-- 시각 측면에서 메시의 각도 및 좌표. rpy = 각도, xyz = 좌표 -->
-      <origin rpy="0.0 0.0 0.0" xyz="0.0 0.0 0.0" />
+      <origin xyz="0 0 0" rpy="0 0 0" />
       <geometry>
-        <!-- 메시 파일 위치 -->
         <mesh filename="package://bumperbot_description/meshes/base_link.STL" />
       </geometry>
     </visual>
     <collision>
-      <origin rpy="0.0 0.0 0.0" xyz="0.0 0.0 0.0" />
+      <origin xyz="0 0 0" rpy="0 0 0" />
       <geometry>
-        <!-- 메시 파일 위치 -->
         <mesh filename="package://bumperbot_description/meshes/base_link.STL" />
       </geometry>
@@ -35,8 +30,7 @@
   </link>
   <joint name="base_joint" type="fixed">
-    <parent link="base_footprint" />
+    <parent link="base_footprint"/>
     <child link="base_link" />
-    <!-- parent에 대한 child의 상대 각도 / 위치 -->
-    <origin rpy="0.0 0.0 0.0" xyz="0.0 0.0 0.033" />
+    <origin xyz="0 0 0.033" rpy="0 0 0"/>
   </joint>
   <link name="wheel_right_link">
@@ -45,30 +39,28 @@
       <mass value="0.0530086090966721" />
       <inertia ixx="1.88176298336665E-05" ixy="-4.8444933029987E-10" ixz="1.88163708851143E-08"
-        iyy="3.11510738647764E-05" iyz="-6.93560663069607E-11" izz="1.8801969558182E-05"
-      />
+               iyy="3.11510738647764E-05" iyz="-6.93560663069607E-11"
+               izz="1.8801969558182E-05" />
     </inertial>
     <visual>
-      <origin rpy="1.57 0 0" xyz="0 0 0" />
+      <origin xyz="0 0 0" rpy="1.57 0 0" />
       <geometry>
         <mesh filename="package://bumperbot_description/meshes/wheel_right_link.STL" />
       </geometry>
     </visual>
-    <!-- collider != mesh -->
     <collision>
-      <origin rpy="1.57 0 0" xyz="0 -0.015 0" />
+      <origin xyz="0 -0.015 0" rpy="1.57 0 0" />
       <geometry>
-        <sphere radius="0.033" />
+        <sphere radius="0.033"/>
       </geometry>
     </collision>
   </link>
-  <!-- continous => rollable -->
   <joint name="wheel_right_joint" type="continuous">
+    <origin xyz="0 -0.0701101849418637 0" rpy="0 0 0" />
     <parent link="base_link" />
     <child link="wheel_right_link" />
-    <!-- y축 -->
     <axis xyz="0 1 0" />
-    <origin rpy="0.0 0.0 0.0" xyz="0.0 -0.07 0.0" />
   </joint>
-  <link name="wheel_left_link">
+  <link
+    name="wheel_left_link">
     <inertial>
       <origin xyz="0 0.014 0" rpy="0 0 0" />
@@ -79,5 +71,5 @@
     </inertial>
     <visual>
-      <origin rpy="-1.57 0 0" xyz="0 0 0" />
+      <origin xyz="0 0 0" rpy="-1.57 0 0" />
       <geometry>
         <mesh filename="package://bumperbot_description/meshes/wheel_left_link.STL" />
@@ -85,24 +77,26 @@
     </visual>
     <collision>
-      <origin rpy="1.57 0 0" xyz="0 0.015 0" />
+      <origin xyz="0 0.015 0" rpy="-1.57 0 0" />
       <geometry>
-        <sphere radius="0.033" />
+        <sphere radius="0.033"/>
       </geometry>
     </collision>
   </link>
-  <!-- continous => rollable -->
   <joint name="wheel_left_joint" type="continuous">
+    <origin xyz="0 0.0701101849418642 0" rpy="0 0 0" />
     <parent link="base_link" />
     <child link="wheel_left_link" />
-    <!-- y축 -->
     <axis xyz="0 1 0" />
-    <origin rpy="0.0 0.0 0.0" xyz="0.0 0.07 0.0" />
   </joint>
   <link name="caster_front_link">
-    <inertia ixx="7.23075276010246E-11" ixy="-6.10956883467859E-16" ixz="2.22849693525031E-15"
+    <inertial>
+      <origin xyz="3.89968128948481E-07 2.40073004698083E-07 0.00219173397061506" rpy="0 0 0" />
+      <mass value="1.44379265037903E-06" />
+      <inertia ixx="7.23075276010246E-11" ixy="-6.10956883467859E-16" ixz="2.22849693525031E-15"
                iyy="3.8713793085917E-11"  iyz="2.93909858781952E-15"
                izz="1.00967486676306E-10" />
+    </inertial>
     <visual>
-      <origin rpy="0.0 0.0 0.0" xyz="0 0 0" />
+      <origin xyz="0 0 0" rpy="0 0 0" />
       <geometry>
         <mesh filename="package://bumperbot_description/meshes/caster_front_link.STL" />
@@ -110,39 +104,44 @@
     </visual>
     <collision>
-      <origin rpy="0 0 0" xyz="0 0 0" />
+      <origin xyz="0 0 0" rpy="0 0 0" />
       <geometry>
-        <sphere radius="0.005" />
+        <sphere radius="0.005"/>
       </geometry>
     </collision>
   </link>
   <joint name="caster_front_joint" type="fixed">
+    <origin xyz="0.04755 0 -0.0275" rpy="0 0 0" />
     <parent link="base_link" />
     <child link="caster_front_link" />
-    <origin rpy="0.0 0.0 0.0" xyz="0.04755 0.0 -0.0275" />
+    <axis xyz="0 0 0" />
   </joint>
   <link name="caster_rear_link">
-    <inertia ixx="7.23075276010246E-11" ixy="-6.10956872363424E-16" ixz="2.22849693527207E-15"
-    iyy="3.87137930859167E-11" iyz="2.939098587861E-15"
-    izz="1.00967486676306E-10" />
+    <inertial>
+      <origin xyz="3.8996812895542E-07 2.40073004698083E-07 0.00219173397061509" rpy="0 0 0" />
+      <mass value="1.44379265037902E-06" />
+      <inertia ixx="7.23075276010246E-11" ixy="-6.10956872363424E-16" ixz="2.22849693527207E-15"
+               iyy="3.87137930859167E-11" iyz="2.939098587861E-15"
+               izz="1.00967486676306E-10" />
+    </inertial>
     <visual>
-      <origin rpy="0.0 0.0 0.0" xyz="0 0 0" />
+      <origin xyz="0 0 0" rpy="0 0 0" />
       <geometry>
         <mesh filename="package://bumperbot_description/meshes/caster_rear_link.STL" />
       </geometry>
     </visual>
-    <!-- visual == volume. not all case. -->
     <collision>
-      <origin rpy="0 0 0" xyz="0 0 0" />
+      <origin xyz="0 0 0" rpy="0 0 0" />
       <geometry>
-        <sphere radius="0.005" />
+        <sphere radius="0.005"/>
       </geometry>
     </collision>
   </link>
   <joint name="caster_rear_joint" type="fixed">
+    <origin xyz="-0.04755 0 -0.0275" rpy="0 0 0" />
     <parent link="base_link" />
     <child link="caster_rear_link" />
-    <origin rpy="0.0 0.0 0.0" xyz="-0.04755 0.0 -0.0275" />
+    <axis xyz="0 0 0" />
   </joint>
-  <link name="can_link">
+   <link name="can_link">
     <visual>
       <origin rpy="1.57 0.0 0.0" xyz="-0.0321 0.0321 0.0" />

File: bumperbot_ws/src/bumperbot_description/urdf/bumperbot_gazebo.xacro (robot description, xacro)
@@ -1,55 +1,49 @@
 <?xml version="1.0"?>
-<robot xmlns:xacro="http://www.ros.org/wiki/xacro" name="bumperbot">
-  <gazebo reference="wheel_right_link">
-    <!-- 마찰력 -->
-    <mu1>100000000000000.0</mu1>
-    <mu2>100000000000000.0</mu2>
+<robot name="bumperbot" xmlns:xacro="http://ros.org/wiki/xacro">
+  <!-- Wheels -->
+  <gazebo reference="wheel_left_link">
+    <mu1>1000000000000000.0</mu1>
+    <mu2>1000000000000000.0</mu2>
     <kp>1000000000000.0</kp>
     <kd>10.0</kd>
-    <!-- simulation solver accuracy -->
     <minDepth>0.001</minDepth>
     <maxVel>0.1</maxVel>
-    <!-- directon of rotation wheel -->
-    <fdirl>1 0 0</fdirl>
+    <fdir1>1 0 0</fdir1>
   </gazebo>
-  <gazebo reference="wheel_left_link">
-    <mu1>100000000000000.0</mu1>
-    <mu2>100000000000000.0</mu2>
+  <gazebo reference="wheel_right_link">
+    <mu1>1000000000000000.0</mu1>
+    <mu2>1000000000000000.0</mu2>
     <kp>1000000000000.0</kp>
     <kd>10.0</kd>
-    <!-- simulation solver accuracy -->
     <minDepth>0.001</minDepth>
     <maxVel>0.1</maxVel>
-    <!-- directon of rotation wheel -->
-    <fdirl>1 0 0</fdirl>
+    <fdir1>1 0 0</fdir1>
   </gazebo>
-  <gazebo reference="caster_front_link">
-    <!-- 시뮬레이션 영향 X -->
+  <!-- Caster Wheels -->
+  <gazebo reference="caster_rear_link">
     <mu1>0.1</mu1>
     <mu2>0.1</mu2>
     <kp>1000000.0</kp>
-    <kd>10.0</kd>
-    <!-- simulation solver accuracy -->
+    <kd>100.0</kd>
     <minDepth>0.001</minDepth>
-    <maxVel>0.1</maxVel>
+    <maxVel>1.0</maxVel>
   </gazebo>
-  <gazebo reference="caster_rear_link">
-    <!-- 시뮬레이션 영향 X -->
+  <gazebo reference="caster_front_link">
     <mu1>0.1</mu1>
     <mu2>0.1</mu2>
     <kp>1000000.0</kp>
-    <kd>10.0</kd>
-    <!-- simulation solver accuracy -->
+    <kd>100.0</kd>
     <minDepth>0.001</minDepth>
-    <maxVel>0.1</maxVel>
+    <maxVel>1.0</maxVel>
   </gazebo>
-  <!-- load proper control library version -->
+  <!-- ROS 2 Control -->
   <gazebo>
-    <!-- ros2 버전에 따라 다른 플러그인을 로드 -->
+    <!-- ROS 2 Humble -->
     <xacro:if value="$(arg is_ignition)">
       <plugin filename="ign_ros2_control-system" name="ign_ros2_control::IgnitionROS2ControlPlugin">
-        <parmeters>$(find bumperbot_controller)/config/bumperbot_controllers.yaml</parmeters>
+        <parameters>$(find bumperbot_controller)/config/bumperbot_controllers.yaml</parameters>
       </plugin>
     </xacro:if>
+    <!-- ROS 2 Iron or above -->
     <xacro:unless value="$(arg is_ignition)">
       <plugin filename="gz_ros2_control-system" name="gz_ros2_control::GazeboSimROS2ControlPlugin">
